File: VBox.kicad_pcb (KiCad board)
At the start: 2 copper layers, 210 x 124.5 mm, 88 parts, among them SW1 SW_Push, SW10 SW_Push, SW11 SW_Push, SW12 SW_Push, SW13 SW_Push, SW14 SW_Push, SW15 SW_Push, SW16 SW_Push, SW17 SW_Push, SW18 SW_Push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

Commit message: text
Other:
- board text added: "Forked from github.com/jfedor2/flatbox"
- board text added: "VBOX"
- board text added: "github.com/CyberVA/vbox"

Commit message: Production files, Gerbers, and adjustments
Parts:
- C1, C10, C4, C8: value 1u -> 1uF
- C11, C12, C13, C14, C15, C16, C5, C6, C7, C9: value 100n -> 100nF
- C2, C3: value 30p -> 30pF
